Commit message: Fixed the discrepancy between the visual and collision origin tags of link_0.

File: robotiq_s_model_visualization/cfg/s-model_finger_articulated_macro.xacro (robot description, xacro)
@@ -19,5 +19,5 @@
 			</visual>
 			<collision>
-				<origin xyz="-0.0455 0.0414 0.036" rpy="0 3.1416 -1.57"/>
+				<origin xyz="0.020 0 0" rpy="0 0 0"/>
 				<geometry>
 					<mesh filename="package://robotiq_s_model_visualization/meshes/s-model_articulated/collision/link_0.STL" />
