Commit message: Correct joint limits for s Model
The upper and lower bounds for the fingers were identified with the
robotiq_joint_state_publisher for the s model and corrected in the
s-model_articulated_macro.xacro for the palm finger joints and in the
s-model_finger_articulated_macro.xacro for the remaining finger joints.

File: robotiq_s_model_visualization/cfg/s-model_articulated_macro.xacro (robot description, xacro)
@@ -37,5 +37,4 @@
 		<!-- end of link list -->
 		<!-- joint list -->
-		<!-- WARNING: LIMITS NOT CORRECT -->
 		<joint name="${prefix}palm_finger_1_joint" type="revolute">
 			<parent link="${prefix}palm"/>
@@ -43,7 +42,6 @@
 			<axis xyz="0 1 0"/>
 			<origin xyz="-0.0455 0.0214 0.036" rpy="0 3.1416 -1.57"/>
-			<limit lower="-0.16" upper="0.25" effort="100" velocity="100"/>
+			<limit lower="-0.1784" upper="0.192" effort="100" velocity="100"/>
 		</joint>
-		<!-- WARNING: LIMITS NOT CORRECT -->
 		<joint name="${prefix}palm_finger_2_joint" type="revolute">
 			<parent link="${prefix}palm"/>
@@ -51,5 +49,5 @@
 			<axis xyz="0 1 0"/>
 			<origin xyz="-0.0455 0.0214 -0.036" rpy="0 3.1416 -1.57"/>
-			<limit lower="-0.25" upper="0.16" effort="100" velocity="100"/>
+			<limit lower="-0.192" upper="0.1784" effort="100" velocity="100"/>
 		</joint>
 		<joint name="${prefix}palm_finger_middle_joint" type="fixed">

File: robotiq_s_model_visualization/cfg/s-model_finger_articulated_macro.xacro (robot description, xacro)
@@ -103,5 +103,4 @@
 		<!-- end of link list -->
 		<!-- joint list -->
-		<!-- WARNING: LIMITS NOT CORRECT -->
 		<joint name="${prefix}joint_1" type="revolute">
 			<parent link="${prefix}link_0"/>
@@ -109,7 +108,6 @@
 			<axis xyz="0 0 1"/>
 			<origin xyz="0.020 0 0" rpy="0 0 0"/>
-			<limit lower="0" upper="3.1416" effort="100" velocity="100"/>
+			<limit lower="0.0495" upper="1.2218" effort="100" velocity="100"/>
 		</joint>
-		<!-- WARNING: LIMITS NOT CORRECT -->
 		<joint name="${prefix}joint_2" type="revolute">
 			<parent link="${prefix}link_1"/>
@@ -117,7 +115,6 @@
 			<axis xyz="0 0 1"/>
 			<origin xyz="0.050 -.028 0" rpy="0 0 -0.52"/>
-			<limit lower="0" upper="3.1416" effort="100" velocity="100"/>
+			<limit lower="0.0" upper="1.5708" effort="100" velocity="100"/>
 		</joint>
-		<!-- WARNING: LIMITS NOT CORRECT -->
 		<joint name="${prefix}joint_3" type="revolute">
 			<parent link="${prefix}link_2"/>
@@ -125,5 +122,5 @@
 			<axis xyz="0 0 1"/>
 			<origin xyz="0.039 0 0" rpy="0 0 0"/>
-			<limit lower="0" upper="3.1416" effort="100" velocity="100"/>
+			<limit lower="-1.2217" upper="-0.0523" effort="100" velocity="100"/>
 		</joint>
 		<!-- end of joint list -->

Commit message: Toolframe for robotiq's s model gripper
New link named tool0.
The toolframe has its origin in the middle of the three fingers, it is
8,75 cm in y direction of the palm link.

A toolframe link is needed as end effector to plan for the hole arm
inclusive the gripper.

File: robotiq_s_model_visualization/cfg/s-model_articulated_macro.xacro (robot description, xacro)
@@ -30,4 +30,5 @@
 			</collision>
 		</link>
+		<link name="${prefix}tool0"/>
         <inertial>
             <origin xyz="0 0 0" rpy="0 0 0"/>
@@ -57,4 +58,9 @@
 			<origin xyz="0.0455 0.0214 0" rpy="0 0 1.57"/>
 		</joint>
+		<joint name="${prefix}palm_tool0" type="fixed">
+			<parent link="${prefix}palm"/>
+			<child link="${prefix}tool0"/>
+			<origin xyz="0.0 0.0875 0.0" rpy="0 0 1.5707"/>
+		</joint>
 		<!-- end of joint list -->
 	</xacro:macro>
