Commit message: add collision mesh & cleanup
- provide the convex hull of the official model as collision model
- fix broken normals in official model (blender: recalculate normals)
- install the meshes folder
- there's no need for a high_res / low_res distinction

File: robotiq_force_torque_sensor/urdf/robotiq_fts150.urdf.xacro (robot description, xacro)
@@ -1,5 +1,5 @@
 <?xml version="1.0"?>
 <robot xmlns:xacro="http://www.ros.org/wiki/xacro" name="robotiq_fts150">
-    <xacro:macro name="robotiq_fts150_hi_res" params="parent prefix *origin">
+    <xacro:macro name="robotiq_fts150" params="parent prefix *origin">
         <!-- mount the fts to the robot -->
         <joint name="{prefix}fts_fix" type="fixed" >
@@ -18,12 +18,12 @@
                 <origin xyz="0 0 0" rpy="0 0 0" />
                 <geometry>
-                    <mesh filename="package://robotiq_force_torque_sensor/models/robotiq_fts150.stl"/>
+                    <mesh filename="package://robotiq_force_torque_sensor/meshes/visual/robotiq_fts150.stl"/>
                 </geometry>
                 <material name="black"/>
             </visual>
             <collision>
-                <origin xyz="0 0 0.01875" rpy="0 0 0" />
+                <origin xyz="0 0 0" rpy="0 0 0" />
                 <geometry>
-                    <cylinder length="0.0375" radius="0.060"/>
+                    <mesh filename="package://robotiq_force_torque_sensor/meshes/collision/robotiq_fts150.stl"/>
                 </geometry>
             </collision>
